Commit message: ompl

File: panda_simulation/franka_description/robots/hand.xacro (robot description, xacro)
@@ -40,5 +40,5 @@
       <inertial>
         <origin xyz="0 0 0" rpy="0 0 0"/>
-        <mass value="0.1"/>
+        <mass value="0.0001"/>
         <inertia ixx="0.1" ixy="0.0" ixz="0.0" iyy="0.1" iyz="0.0" izz="0.1"/>
       </inertial>
@@ -59,5 +59,5 @@
       <inertial>
         <origin xyz="0 0 0" rpy="0 0 0"/>
-        <mass value="0."/>
+        <mass value="0.0001"/>
         <inertia ixx="0.1" ixy="0.0" ixz="0.0" iyy="0.1" iyz="0.0" izz="0.1"/>
       </inertial>
@@ -78,5 +78,5 @@
       <mimicjoint="${ns}_finger_joint1" />
     </joint>
- -->
+-->
     <link name="virtual_link">
       <inertial>

File: panda_simulation/franka_description/robots/panda.transmission.xacro (robot description, xacro)
@@ -89,13 +89,12 @@
                 <mechanicalReduction>1</mechanicalReduction>
             </actuator>
-        </transmission>  -->
-<!--
+        </transmission>
             <transmission name="${robot_name}_leftfinger">
                 <type>transmission_interface/SimpleTransmission</type>
                 <joint name="${robot_name}_finger_joint1">
-                    <hardwareInterface>hardware_interface/EffortJointInterface</hardwareInterface>
+                    <hardwareInterface>hardware_interface/PositionJointInterface</hardwareInterface>
                 </joint>
                 <actuator name="${robot_name}_finger_joint1">
-                    <hardwareInterface>hardware_interface/EffortJointInterface</hardwareInterface>
+                    <hardwareInterface>hardware_interface/PositionJointInterface</hardwareInterface>
                     <mechanicalReduction>1</mechanicalReduction>
                 </actuator>
@@ -104,12 +103,12 @@
                 <type>transmission_interface/SimpleTransmission</type>
                 <joint name="${robot_name}_finger_joint2">
-                    <hardwareInterface>hardware_interface/EffortJointInterface</hardwareInterface>
+                    <hardwareInterface>hardware_interface/PositionJointInterface</hardwareInterface>
                 </joint>
                 <actuator name="${robot_name}_finger_joint2">
-                    <hardwareInterface>hardware_interface/EffortJointInterface</hardwareInterface>
+                    <hardwareInterface>hardware_interface/PositionJointInterface</hardwareInterface>
                     <mechanicalReduction>1</mechanicalReduction>
                 </actuator>
             </transmission>
--->
+ -->
     </xacro:macro>
 </robot>

Commit message: gripper

File: panda_simulation/franka_description/robots/hand.xacro (robot description, xacro)
@@ -26,5 +26,5 @@
       </inertial>
     </link>
-<!--
+<!--  -->
     <link name="${ns}_leftfinger">
       <visual>
@@ -40,5 +40,5 @@
       <inertial>
         <origin xyz="0 0 0" rpy="0 0 0"/>
-        <mass value="0.0001"/>
+        <mass value="0.01"/>
         <inertia ixx="0.1" ixy="0.0" ixz="0.0" iyy="0.1" iyz="0.0" izz="0.1"/>
       </inertial>
@@ -63,4 +63,5 @@
       </inertial>
     </link>
+ <!-- -->
     <joint name="${ns}_finger_joint1" type="prismatic">
       <parent link="${ns}_hand"/>
@@ -76,7 +77,5 @@
       <axis xyz="0 -1 0"/>
       <limit effort="20" lower="0.0" upper="0.04" velocity="0.2"/>
-      <mimicjoint="${ns}_finger_joint1" />
     </joint>
--->
     <link name="virtual_link">
       <inertial>

File: panda_simulation/franka_description/robots/panda.transmission.xacro (robot description, xacro)
@@ -90,25 +90,24 @@
             </actuator>
         </transmission>
-            <transmission name="${robot_name}_leftfinger">
+                    <hardwareInterface>hardware_interface/EffortJointInterface</hardwareInterface>
+-->
+           <transmission name="${robot_name}_trans_rightfinger">
                 <type>transmission_interface/SimpleTransmission</type>
                 <joint name="${robot_name}_finger_joint1">
-                    <hardwareInterface>hardware_interface/PositionJointInterface</hardwareInterface>
+                    <hardwareInterface>hardware_interface/EffortJointInterface</hardwareInterface>
                 </joint>
                 <actuator name="${robot_name}_finger_joint1">
-                    <hardwareInterface>hardware_interface/PositionJointInterface</hardwareInterface>
                     <mechanicalReduction>1</mechanicalReduction>
                 </actuator>
             </transmission>
-            <transmission name="${robot_name}_rightfinger">
+            <transmission name="${robot_name}_trans_leftfinger">
                 <type>transmission_interface/SimpleTransmission</type>
                 <joint name="${robot_name}_finger_joint2">
-                    <hardwareInterface>hardware_interface/PositionJointInterface</hardwareInterface>
+                    <hardwareInterface>hardware_interface/EffortJointInterface</hardwareInterface>
                 </joint>
                 <actuator name="${robot_name}_finger_joint2">
-                    <hardwareInterface>hardware_interface/PositionJointInterface</hardwareInterface>
                     <mechanicalReduction>1</mechanicalReduction>
                 </actuator>
             </transmission>
- -->
     </xacro:macro>
 </robot>

File: panda_simulation/franka_description/robots/panda_arm_world.urdf.xacro (robot description, xacro)
@@ -9,5 +9,4 @@
   <xacro:include filename="$(find franka_description)/robots/panda.gazebo.xacro"/>
   <xacro:include filename="$(find franka_description)/robots/panda.transmission.xacro"/>
-  <xacro:include filename="$(find franka_description)/robots/plugin.xacro"/>
   <!-- Robot arm definition-->
   <xacro:panda_arm />

Commit message: window

File: panda_simulation/franka_description/robots/hand.xacro (robot description, xacro)
@@ -40,5 +40,5 @@
       <inertial>
         <origin xyz="0 0 0" rpy="0 0 0"/>
-        <mass value="0.01"/>
+        <mass value="0.001"/>
         <inertia ixx="0.1" ixy="0.0" ixz="0.0" iyy="0.1" iyz="0.0" izz="0.1"/>
       </inertial>
@@ -59,5 +59,5 @@
       <inertial>
         <origin xyz="0 0 0" rpy="0 0 0"/>
-        <mass value="0.0001"/>
+        <mass value="0.001"/>
         <inertia ixx="0.1" ixy="0.0" ixz="0.0" iyy="0.1" iyz="0.0" izz="0.1"/>
       </inertial>

File: panda_simulation/franka_description/robots/panda_arm_world.urdf.xacro (robot description, xacro)
@@ -9,4 +9,5 @@
   <xacro:include filename="$(find franka_description)/robots/panda.gazebo.xacro"/>
   <xacro:include filename="$(find franka_description)/robots/panda.transmission.xacro"/>
+  <xacro:include filename="$(find franka_description)/robots/hand_attachment.xacro"/>
   <!-- Robot arm definition-->
   <xacro:panda_arm />
@@ -15,3 +16,5 @@
   <xacro:panda_gazebo robot_name="$(arg robot_name)" />
   <xacro:panda_transmission robot_name="$(arg robot_name)" />
+  <!-- Attachment -->
+  <xacro:stick_urdf parent="virtual_link" />
 </robot>
